File: hardware/adc-frontend/layouts/default/default.kicad_pcb (KiCad board)
At the start: 2 copper layers, 120 x 90 mm, 107 parts

Commit message: ネットクラス+差動ペア設定(GbE/Power/Analog_RGB/Clock)
レイアウト指示書§2に基づき default.kicad_pro に4ネットクラスを定義しパターン割当:
- GbE_diff: track0.2/clr0.4/DP幅0.2/DPギャップ0.2(100Ω暫定・要スタックアップ調整) → eth1_*/eth2_*
- Power: track0.4/clr0.2/via0.8 → power_5v*/p5v_ext/p3v3_*/p1v9_*
- Analog_RGB: track0.25/clr0.30 → c_ac-power-*/c_sog3-power-*
- Clock: track0.25/clr0.25 → dataclk/ext_clk/audio_mclk/bck/lrck

差動ペア認識のためGbEネットを大文字_P/_N接尾辞へ改名(eth1_1p→eth1_1_P等、
mech.ato HeaderP1定義+main.ato接続)。KiCadの差動ペアルータ/DRCは+/-またはP/N
(大文字)接尾辞のみ認識するため。8ペア完全成立を確認。

検証: ato build成功、atopileは.kicad_proを上書きしない、fnmatchでパターン網羅確認
(GbE16/Power8/Analog_RGB7/Clock5本)、kicad-cli drcでプロジェクト+ネットクラスが
解析エラー無くロード(違反はすべて未配線/粗配置由来でネットクラス起因ゼロ)。

Co-Authored-By: Claude Opus 4.8 (1M context) <noreply@anthropic.com>
Claude-Session: https://claude.ai/code/session_01J5hbhQ5HHukYPsP5Uq7b5N
Connections:
- net eth1_1n renamed eth1_1_N
- net eth1_1p renamed eth1_1_P
- net eth1_2n renamed eth1_2_N
- net eth1_2p renamed eth1_2_P
- net eth1_3n renamed eth1_3_N
- net eth1_3p renamed eth1_3_P
- net eth1_4n renamed eth1_4_N
- net eth1_4p renamed eth1_4_P
- net eth2_1n renamed eth2_1_N
- net eth2_1p renamed eth2_1_P
- net eth2_2n renamed eth2_2_N
- net eth2_2p renamed eth2_2_P
- net eth2_3n renamed eth2_3_N
- net eth2_3p renamed eth2_3_P
- net eth2_4n renamed eth2_4_N
- net eth2_4p renamed eth2_4_P
Changed lines of the file:
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@@
 	(net 147 "B8")
 	(net 94 "ct_caps[1]-power-hv")
-	(net 95 "eth2_3n")
-	(net 100 "eth2_3p")
-	(net 148 "eth1_4n")
-	(net 149 "eth1_2p")
-	(net 150 "eth1_4p")
-	(net 151 "eth2_2p")
-	(net 152 "eth2_4p")
-	(net 153 "eth2_2n")
-	(net 154 "eth2_4n")
-	(net 155 "eth2_1n")
+	(net 95 "eth2_3_N")
+	(net 100 "eth2_3_P")
+	(net 148 "eth1_4_N")
+	(net 149 "eth1_2_P")
+	(net 150 "eth1_4_P")
+	(net 151 "eth2_2_P")
+	(net 152 "eth2_4_P")
+	(net 153 "eth2_2_N")
+	(net 154 "eth2_4_N")
+	(net 155 "eth2_1_N")
 	(net 156 "ct_caps[0]-power-hv")
-	(net 157 "eth2_1p")
+	(net 157 "eth2_1_P")
 	(net 158 "chassis")
-	(net 159 "eth1_1p")
-	(net 160 "eth1_1n")
-	(net 161 "eth1_3p")
-	(net 162 "eth1_3n")
-	(net 163 "eth1_2n")
+	(net 159 "eth1_1_P")
+	(net 160 "eth1_1_N")
+	(net 161 "eth1_3_P")
+	(net 162 "eth1_3_N")
+	(net 163 "eth1_2_N")
 	(net 1 "c_in_l-power-hv-1")
 	(net 2 "c_in_r-power-hv-1")
@@
 			(layers "*.Cu" "*.Mask")
 			(remove_unused_layers no)
-			(net 151 "eth2_2p")
+			(net 151 "eth2_2_P")
 		)
 		(pad "6" thru_hole oval
@@
 			(layers "*.Cu" "*.Mask")
 			(remove_unused_layers no)
-			(net 152 "eth2_4p")
+			(net 152 "eth2_4_P")
 		)
 		(pad "7" thru_hole oval
@@
 			(layers "*.Cu" "*.Mask")
 			(remove_unused_layers no)
-			(net 153 "eth2_2n")
+			(net 153 "eth2_2_N")
 		)
 		(pad "8" thru_hole oval
@@
 			(layers "*.Cu" "*.Mask")
 			(remove_unused_layers no)
-			(net 154 "eth2_4n")
+			(net 154 "eth2_4_N")
 		)
 		(pad "9" thru_hole oval
@@
 			(layers "*.Cu" "*.Mask")
 			(remove_unused_layers no)
-			(net 155 "eth2_1n")
+			(net 155 "eth2_1_N")
 		)
 		(pad "10" thru_hole oval
@@
 			(layers "*.Cu" "*.Mask")
 			(remove_unused_layers no)
-			(net 95 "eth2_3n")
+			(net 95 "eth2_3_N")
 		)
 		(pad "11" thru_hole oval
@@
 			(layers "*.Cu" "*.Mask")
 			(remove_unused_layers no)
-			(net 157 "eth2_1p")
+			(net 157 "eth2_1_P")
 		)
 		(pad "12" thru_hole oval
@@
 			(layers "*.Cu" "*.Mask")
 			(remove_unused_layers no)
-			(net 100 "eth2_3p")
+			(net 100 "eth2_3_P")
 		)
 		(pad "13" thru_hole oval
@@
 			(layers "*.Cu" "*.Mask")
 			(remove_unused_layers no)
-			(net 159 "eth1_1p")
+			(net 159 "eth1_1_P")
 		)
 		(pad "24" thru_hole oval
@@
 			(layers "*.Cu" "*.Mask")
 			(remove_unused_layers no)
-			(net 161 "eth1_3p")
+			(net 161 "eth1_3_P")
 		)
 		(pad "25" thru_hole oval
@@
 			(layers "*.Cu" "*.Mask")
 			(remove_unused_layers no)
-			(net 160 "eth1_1n")
+			(net 160 "eth1_1_N")
 		)
 		(pad "26" thru_hole oval
@@
 			(layers "*.Cu" "*.Mask")
 			(remove_unused_layers no)
-			(net 162 "eth1_3n")
+			(net 162 "eth1_3_N")
 		)
 		(pad "27" thru_hole oval
@@
 			(layers "*.Cu" "*.Mask")
 			(remove_unused_layers no)
-			(net 163 "eth1_2n")
+			(net 163 "eth1_2_N")
 		)
 		(pad "28" thru_hole oval
@@
 			(layers "*.Cu" "*.Mask")
 			(remove_unused_layers no)
-			(net 148 "eth1_4n")
+			(net 148 "eth1_4_N")
 		)
 		(pad "29" thru_hole oval
@@
 			(layers "*.Cu" "*.Mask")
 			(remove_unused_layers no)
-			(net 149 "eth1_2p")
+			(net 149 "eth1_2_P")
 		)
 		(pad "30" thru_hole oval
@@
 			(layers "*.Cu" "*.Mask")
 			(remove_unused_layers no)
-			(net 150 "eth1_4p")
+			(net 150 "eth1_4_P")
 		)
 		(embedded_fonts no)
@@
 			(drill 0.9099804)
 			(layers "*.Cu" "*.Mask")
-			(net 157 "eth2_1p")
+			(net 157 "eth2_1_P")
 		)
 		(pad "P3" thru_hole circle
@@
 			(drill 0.9099804)
 			(layers "*.Cu" "*.Mask")
-			(net 155 "eth2_1n")
+			(net 155 "eth2_1_N")
 		)
 		(pad "P4" thru_hole circle
@@
 			(drill 0.9099804)
 			(layers "*.Cu" "*.Mask")
-			(net 151 "eth2_2p")
+			(net 151 "eth2_2_P")
 		)
 		(pad "P5" thru_hole circle
@@
 			(drill 0.9099804)
 			(layers "*.Cu" "*.Mask")
-			(net 100 "eth2_3p")
+			(net 100 "eth2_3_P")
 		)
 		(pad "P6" thru_hole circle
@@
 			(drill 0.9099804)
 			(layers "*.Cu" "*.Mask")
-			(net 95 "eth2_3n")
+			(net 95 "eth2_3_N")
 		)
 		(pad "P7" thru_hole circle
@@
 			(drill 0.9099804)
 			(layers "*.Cu" "*.Mask")
-			(net 153 "eth2_2n")
+			(net 153 "eth2_2_N")
 		)
 		(pad "P8" thru_hole circle
@@
 			(drill 0.9099804)
 			(layers "*.Cu" "*.Mask")
-			(net 152 "eth2_4p")
+			(net 152 "eth2_4_P")
 		)
 		(pad "SHIELD1" thru_hole circle
@@
 			(drill 0.9099804)
 			(layers "*.Cu" "*.Mask")
-			(net 154 "eth2_4n")
+			(net 154 "eth2_4_N")
 		)
 		(pad "P10" thru_hole circle
@@
 			(drill 0.9099804)
 			(layers "*.Cu" "*.Mask")
-			(net 159 "eth1_1p")
+			(net 159 "eth1_1_P")
 		)
 		(pad "P3" thru_hole circle
@@
 			(drill 0.9099804)
 			(layers "*.Cu" "*.Mask")
-			(net 160 "eth1_1n")
+			(net 160 "eth1_1_N")
 		)
 		(pad "P4" thru_hole circle
@@
 			(drill 0.9099804)
 			(layers "*.Cu" "*.Mask")
-			(net 149 "eth1_2p")
+			(net 149 "eth1_2_P")
 		)
 		(pad "P5" thru_hole circle
@@
 			(drill 0.9099804)
 			(layers "*.Cu" "*.Mask")
-			(net 161 "eth1_3p")
+			(net 161 "eth1_3_P")
 		)
 		(pad "P6" thru_hole circle
@@
 			(drill 0.9099804)
 			(layers "*.Cu" "*.Mask")
-			(net 162 "eth1_3n")
+			(net 162 "eth1_3_N")
 		)
 		(pad "P7" thru_hole circle
@@
 			(drill 0.9099804)
 			(layers "*.Cu" "*.Mask")
-			(net 163 "eth1_2n")
+			(net 163 "eth1_2_N")
 		)
 		(pad "P8" thru_hole circle
@@
 			(drill 0.9099804)
 			(layers "*.Cu" "*.Mask")
-			(net 150 "eth1_4p")
+			(net 150 "eth1_4_P")
 		)
 		(pad "SHIELD1" thru_hole circle
@@
 			(drill 0.9099804)
 			(layers "*.Cu" "*.Mask")
-			(net 148 "eth1_4n")
+			(net 148 "eth1_4_N")
 		)
 		(pad "P10" thru_hole circle

Commit message: 4層化+JLC04161H-7628スタックアップ設定, GbE差動ギャップを100Ω値へ, カスタムDRC追加
- 基板を2層→4層化(L1信号/L2=In1.Cu GNDプレーン/L3=In2.Cu PWRプレーン/L4信号)。
  physical stackupをJLCPCB JLC04161H-7628相当に設定(上部プリプレグ7628=0.2104mm/εr4.6、
  コア1.065mm、内層0.5oz/外層1oz、板厚1.6mm、ENIG)。上部を厚い7628にしてGbE 100Ωを
  実用トレース幅で引けるように。ato buildがスタックアップを保持することを検証済み。
- GbE_diff 差動ギャップ 0.20→0.13mm(このスタックアップでのエッジ結合μストリップ解析≈100Ω)。
  最終値はJLC/KiCad内蔵インピーダンス計算で要確認(スタックアップ設定済みで即計算可)。
- カスタムDRC default.kicad_dru 追加: GbEペア内スキュー≤0.15mm/非結合≤5mm/ビア≤2/
  対他ネットクリアランス≥0.6mm、クロックビア≤3。kicad-cli drcで解析エラー無しを確認。
- 指示書§0/§2を実装状態へ更新。

Co-Authored-By: Claude Opus 4.8 (1M context) <noreply@anthropic.com>
Claude-Session: https://claude.ai/code/session_01J5hbhQ5HHukYPsP5Uq7b5N
Other:
- copper layers 2 -> 4

Commit message: main.ato改修: SO-DIMM化 + オンボードFT2232H書換え経路
- Colorlight i5をDDR2 SO-DIMM 200Pソケット(SoDimmI5)へ直挿し化。
  旧EXT P2/P4/P1ヘッダを廃止し全GPIO/ETH/電源をSO-DIMMピンへ移設。
- FT2232H(C27882)搭載: USB-C(J10)1本で電源+書換えを兼用。
  ch.A MPSSE=JTAG(openFPGALoader -c ft2232, メイン経路)、ch.B=UART。
  EEPROM 93LC56(C6164)+12MHz水晶(C9002)+内部1.8V LDOでコア給電。
- JTAG: ポゴピン4本(PogoPin)でi5底面パッド(TCK/TMS/TDI/TDO)へバネ接触。
  加えて念のためのDNPヘッダ(HeaderJtag 1x6, コネクタ未実装)を並列引き出し。
- GbEリンクLED: 主ポート(ETH2)緑/黄をFPGA GPIO(io_r1/io_t1)+R220で駆動。
- 新規パッシブ: R10K(nRESET)/R12K(REF基準)/C33pF(水晶負荷)。
- PHYインデックス表記を修正: ETH2=PHY0=litex eth1(映像既定)で統一。

ato build 全ターゲット成功。ネットリスト結線をSO-DIMM(200pad)/FT2232H/JTAG
(ポゴ+ヘッダ並列)/UART/LEDについて検証済み。手実装/DNP部品(ソケット・ポゴ・
JTAGヘッダ)はBOMから除外。

Co-Authored-By: Claude Opus 4.8 (1M context) <noreply@anthropic.com>
Claude-Session: https://claude.ai/code/session_01J5hbhQ5HHukYPsP5Uq7b5N
Parts:
- removed J3, J4: , _mech:Header_2x15_P2.54mm
- added C45: {ℝ+}F, SAMSUNG_CL05B104KO5NNNC:C0402, F.Cu at (200.0, 0.00)
- added C46: {ℝ+}F, SAMSUNG_CL10C330JB8NNNC:C0603, F.Cu at (170.0, 0.00)
- added C63: {ℝ+}F, SAMSUNG_CL10C330JB8NNNC:C0603, F.Cu at (180.0, 0.00)
- added C64: {ℝ+}F, SAMSUNG_CL05B104KO5NNNC:C0402, F.Cu at (30.0, 0.00)
- added C65: {ℝ+}F, SAMSUNG_CL05B104KO5NNNC:C0402, F.Cu at (40.0, 0.00)
- added C66: {ℝ+}F, SAMSUNG_CL05B104KO5NNNC:C0402, F.Cu at (50.0, 0.00)
- added C67: {ℝ+}F, SAMSUNG_CL05B104KO5NNNC:C0402, F.Cu at (60.0, 0.00)
- added C68: {ℝ+}F, SAMSUNG_CL05B104KO5NNNC:C0402, F.Cu at (110.0, 0.00)
- added C69: {ℝ+}F, SAMSUNG_CL05B104KO5NNNC:C0402, F.Cu at (120.0, 0.00)
- added C70: {ℝ+}F, SAMSUNG_CL05B104KO5NNNC:C0402, F.Cu at (130.0, 0.00)
- added C71: {ℝ+}F, SAMSUNG_CL21A106KAYNNNE:C0805, F.Cu at (80.0, 0.00)
- added C72: {ℝ+}F, SAMSUNG_CL05B104KO5NNNC:C0402, F.Cu at (70.0, 0.00)
- added C73: {ℝ+}F, SAMSUNG_CL10A105KB8NNNC:C0603, F.Cu at (100.0, 0.00)
- added C74: {ℝ+}F, SAMSUNG_CL05B104KO5NNNC:C0402, F.Cu at (90.0, 0.00)
- added FB4: , TDK_MPZ1608S221ATA00:L0603, F.Cu at (10.0, 0.00)
- added FB5: , TDK_MPZ1608S221ATA00:L0603, F.Cu at (20.0, 0.00)
- added PG1: , _mech:PogoPin_D1.0mm, F.Cu at (0.00, 0.00)
- added PG2: , _mech:PogoPin_D1.0mm, F.Cu at (20.0, 0.00)
- added PG3: , _mech:PogoPin_D1.0mm, F.Cu at (30.0, 0.00)
- added PG4: , _mech:PogoPin_D1.0mm, F.Cu at (10.0, 0.00)
- added R14: {ℝ+}Ω, UNI_ROYAL_0402WGF1202TCE:R0402, F.Cu at (140.0, 0.00)
- added R15: {ℝ+}Ω, UNI_ROYAL_0402WGF1002TCE:R0402, F.Cu at (150.0, 0.00)
- added R16: {ℝ+}Ω, UNI_ROYAL_0402WGF2200TCE:R0402, F.Cu at (10.0, 0.00)
- added R17: {ℝ+}Ω, UNI_ROYAL_0402WGF2200TCE:R0402, F.Cu at (20.0, 0.00)
- added U11: , JST_DM_7D4_H2500_M:DIMM-SMD_DM-7D4-H2500-M, F.Cu at (0.00, 0.00)
- added U12: , MICROCHIP_93LC56BT_I_SN:SOIC-8_L4.9-W3.9-P1.27-LS6.0-BL, F.Cu at (190.0, 0.00)
- added U13: , FTDI_FT2232HL_REEL:LQFP-64_L10.0-W10.0-P0.50-LS12.0-TL, F.Cu at (0.00, 0.00)
- added X3: , YXC_X322512MSB4SI:CRYSTAL-SMD_4P-L3.2-W2.5-BL, F.Cu at (160.0, 0.00)
- J1: footprint _mech:Header_2x15_P2.54mm -> _mech:Header_1x6_P2.54mm
- moved J1 129.3 mm to (0.00, 0.00)
Connections:
- net 43 renamed tvp-43
- net 44 renamed tvp-44
- net 55 renamed tvp-55
- J1 pad 1: 1 -> jtag_tck
- J1 pad 2: 1 -> jtag_tms
- J1 pad 3: gnd -> jtag_tdi
- J1 pad 4: gnd -> jtag_tdo
- J1 pad 5: eth2_2_P -> gnd
- J1 pad 6: eth2_4_P -> p3v3_io-hv
- J11 pad 12: eth.jack2-led_g_k -> led_g_k
- J11 pad 13: eth.jack2-led_y_k -> led_y_k
- J2 pad 12: led_g_k -> gnd
- J2 pad 13: led_y_k -> gnd
- U10 pad 23: 23-1 -> vsout
- U10 pad 25: 25-1 -> sogout
- U10 pad 31: 13-2 -> 140
- U10 pad 32: 11 -> 136
- U10 pad 33: 33 -> 128
- U10 pad 34: 34 -> 153
- U10 pad 35: 26 -> 35
- U10 pad 36: 25 -> 36
- U10 pad 37: 24 -> 37
- U10 pad 38: 23 -> 38
- U10 pad 45: 22 -> 45-1
- U10 pad 46: 21 -> 46-1
- U10 pad 47: 20 -> 47
- U10 pad 48: 19 -> 48-1
- U10 pad 49: 18-1 -> 49
- U10 pad 50: 17-1 -> 50
- U10 pad 51: 14-1 -> 51
- U10 pad 52: 13-1 -> 52-1
- U10 pad 57: 57 -> 57-1
- U10 pad 58: 58 -> 58-1
- U10 pad 59: 59 -> 59-1
- U10 pad 61: 5 -> 61
- U10 pad 62: 4-1 -> 62
- U10 pad 63: 3 -> 63
- U10 pad 64: 2 -> 64
- U10 pad 65: 1-1 -> 65

Commit message: レイアウト: 手動配線の現状を保存 + 主要ネットを明示命名
- main.ato: override_net_nameで機能上重要なネットに固定名を付与
  (アナログRGB vin_*/rin3/gin3/bin3/sogin3, デジタル映像バス vd_*,
   avdd/pll_avdd, PLLフィルタ, 同期, 音声, 未使用終端 *_nc)
- default.kicad_pro: netclassパターンを新名に追従(Analog_RGB/Power)
- default.kicad_pcb/.prl: 手動レイアウト作業の途中状態を保存

Co-Authored-By: Claude Opus 4.8 (1M context) <noreply@anthropic.com>
Parts:
- moved U13 198.1 mm to (114.9, 161.3)
- moved J1 196.3 mm to (92.1, 173.4)
- moved U11 189.9 mm to (153.0, 112.4), turned to 180 degrees
- moved U12 165.9 mm to (113.7, 147.3)
- moved U9 162.6 mm to (95.7, 153.4), turned to 180 degrees
- moved J9 162.1 mm to (76.0, 162.6), turned to -90 degrees
- moved J7 155.7 mm to (77.4, 150.1)
- moved U7 153.6 mm to (95.9, 146.1), turned to 180 degrees
- moved J5 146.0 mm to (168.3, 149.9)
- moved U6 142.8 mm to (154.9, 68.6)
- moved J8 123.9 mm to (76.1, 131.4), turned to -90 degrees
- moved J6 113.4 mm to (74.7, 119.3), turned to 90 degrees
- moved C7 113.1 mm to (94.0, 133.3)
- moved U2 111.5 mm to (100.3, 129.9), turned to 90 degrees
- moved C8 110.8 mm to (93.9, 131.4)
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Connections:
- net 128 renamed vd_b4
- net 136 renamed vd_b3
- net 140 renamed vd_b2
- net 153 renamed vd_b5
- net 35 renamed vd_b6
- net 36 renamed vd_b7
- net 37 renamed vd_b8
- net 38 renamed vd_b9
- net 45-1 renamed vd_g2
- net 46-1 renamed vd_g3
- net 47 renamed vd_g4
- net 48-1 renamed vd_g5
- net 49 renamed vd_g6
- net 50 renamed vd_g7
- net 51 renamed vd_g8
- net 52-1 renamed vd_g9
- net 57-1 renamed vd_r2
- net 58-1 renamed vd_r3
- net 59-1 renamed vd_r4
- net 61 renamed vd_r5
- net 62 renamed vd_r6
- net 63 renamed vd_r7
- net 64 renamed vd_r8
- net 65 renamed vd_r9
- net 87 renamed pll_filt1
- net c_ac-power-hv renamed vin_r
- net c_ac-power-hv-1 renamed vin_b
- net c_ac-power-lv renamed bin3
- net c_ac-power-lv-1 renamed gin3
- net c_ac-power-lv-2 renamed rin3
- net c_filt1-power-hv renamed pll_filt_mid
- net c_filt2-power-hv renamed pll_filt2
- net c_filt2-power-lv renamed pll_f
- net c_in_l-power-hv renamed aud_dsub_l
- net c_in_l-power-hv-1 renamed aud_line_l
- net c_in_l-power-lv renamed aud_dsub_l_ac
- net c_in_l-power-lv-1 renamed aud_line_l_ac
- net c_in_r-power-hv renamed aud_dsub_r
- net c_in_r-power-hv-1 renamed aud_line_r
- net c_in_r-power-lv renamed aud_line_r_ac
- net c_sog3-power-hv renamed vin_g
- net c_sog3-power-lv renamed sogin3
- net c_vref_b-power-hv renamed aud_vref_dsub
- net c_vref_b-power-hv-1 renamed aud_vref_line
- net c_vs-power-hv renamed vsync_delayed
- net dec_caps[5]-power-hv renamed avdd
- net dec_caps[7]-power-hv renamed pll_avdd
- net dout renamed i2s_dout_dsub
- net dout-1 renamed i2s_dout_line
- net lv renamed aud_dsub_r_ac
- net nc_caps[0]-power-hv renamed rin1_nc
- net nc_caps[1]-power-hv renamed rin2_nc
- net nc_caps[2]-power-hv renamed bin1_nc
- net nc_caps[3]-power-hv renamed bin2_nc
- net nc_caps[4]-power-hv renamed gin1_nc
- net nc_caps[5]-power-hv renamed gin2_nc
- net nc_caps[6]-power-hv renamed gin4_nc
- net nc_sog_caps[0]-power-hv renamed sogin1_nc
- net nc_sog_caps[1]-power-hv renamed sogin2_nc
- net out_b renamed vsync_a
Routing:
- net vin_g: track 0.00 -> 2.75 mm
- net vin_r: track 0.00 -> 1.27 mm
- added copper zone on F.Cu, net gnd
Other:
- board size 120 x 90 mm -> 142.2 x 111.6 mm
